File: rp2040-board.kicad_pcb (KiCad board)
At the start: 2 copper layers, 23 x 39 mm, 39 parts, among them CN1 HX JN1.27-2X5 TP H4.9, J1 USB_C_Receptacle_USB2.0_14P, SW1 TS-1088-AR02016, SW2 TS-1088-AR02016, U1 W25Q128JVSIQTR, U2 USBLC6-2SC6, U3 LM3940IMP-3.3/NOPB, U4 RP2040, Y1 ABM8-272-T3_C20625731

Commit message: Hopefully finished routing
Parts:
- removed R9: 10Kohm, Resistor_SMD:R_0402_1005Metric
- added C18: 0.1uf, Capacitor_SMD:C_0402_1005Metric, F.Cu at (140.6, 98.8)
- C11: value 0.1uf -> 15pf
- C13: value 1uf -> 0.1uf
- C15: value 0.1uf -> 1uf
- C3: value 22uf -> 0.1uf; footprint Capacitor_SMD:C_0603_1608Metric -> Capacitor_SMD:C_0402_1005Metric
- C4: value 0.1uf -> 22uf; footprint Capacitor_SMD:C_0402_1005Metric -> Capacitor_SMD:C_0603_1608Metric
- C9: value 15pf -> 0.1uf
- CN1: value HX JN1.27-2X5 TP H4.9 -> SM04B-SRSS-TB; footprint easyeda2kicad:IDC-SMD_10P-P1.27-3220-10-0300-00 -> easyeda2kicad:CONN-SMD_4P-P1.00_SM04B-SRSS-TB-LF-SN
- J1: footprint Connector_USB:USB_C_Receptacle_GCT_USB4105-xx-A_16P_TopMnt_Horizontal -> Connector_USB:USB_C_Receptacle_HRO_TYPE-C-31-M-12
- LED1: value 0603White light_C2290 -> SK6812MINI-E_C5149201; footprint easyeda2kicad:LED0603-R-RD_WHITE -> easyeda2kicad:LED-SMD_4P-L3.2-W2.8-LS5.9_SK6812MINI-E
- R8: value 330Ohm -> 10Kohm; footprint Resistor_SMD:R_0603_1608Metric -> Resistor_SMD:R_0402_1005Metric
- U3: value LM3940IMP-3.3/NOPB -> AMS1117-3.3; footprint easyeda2kicad:SOT-223_L6.5-W3.5-P2.30-LS7.0-BR -> easyeda2kicad:SOT-223-3_L6.5-W3.4-P2.30-LS7.0-BR
- moved C2 63.1 mm to (135.3, 84.2), turned to 180 degrees
- moved C4 62.4 mm to (131.4, 91.8), turned to -90 degrees
- moved R4 62.3 mm to (142.0, 93.8), turned to -90 degrees
- moved C1 58.8 mm to (133.2, 91.5), turned to 180 degrees
- moved LED1 58.4 mm to (134.2, 112.8), turned to -135 degrees
- moved C16 56.3 mm to (142.6, 98.8), turned to 90 degrees
- moved R3 55.6 mm to (148.2, 93.8), turned to -90 degrees
- moved C12 54.8 mm to (141.6, 98.8), turned to 90 degrees
- moved C5 52.3 mm to (136.6, 104.2), turned to -90 degrees
- moved C15 51.9 mm to (146.6, 98.8), turned to 90 degrees
- moved C6 51.3 mm to (136.6, 106.2), turned to 90 degrees
- moved C13 50.3 mm to (148.6, 98.8), turned to 90 degrees
- moved C14 50.0 mm to (147.6, 98.8), turned to 90 degrees
- moved C10 49.4 mm to (138.8, 114.5), turned to -90 degrees
- moved C17 48.9 mm to (145.3, 111.4)
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Connections:
- C10 pad 1: Net-(C10-Pad1) -> /XIN
- C11 pad 1: +3V3 -> Net-(C11-Pad1)
- C14 pad 1: +1V1 -> +3V3
- C15 pad 1: +3V3 -> +1V1
- C16 pad 1: +1V1 -> +3V3
- C3 pad 1: +3V3 -> GND
- C3 pad 2: GND -> +3V3
- C9 pad 1: /XIN -> +3V3
- CN1 pad 1: +3V3 -> GND
- CN1 pad 2: /SWDIO -> +3V3
- CN1 pad 3: GND -> /GPIO16
- CN1 pad 4: /SWCLK -> /GPIO17
- CN1 pad 6: unconnected-(CN1-Pad6) -> GND
- J2 pad 1: /RST -> +3V3
- J2 pad 10: /GPIO25 -> /GPIO08
- J2 pad 11: /GPIO26 -> /GPIO09
- J2 pad 12: /GPIO27 -> /GPIO10
- J2 pad 13: /GPIO28 -> /GPIO11
- J2 pad 14: /GPIO29 -> /GPIO12
- J2 pad 15: GND -> /GPIO13
- J2 pad 16: /VSYS -> GND
- J2 pad 2: /SWCLK -> GND
- J2 pad 3: /SWDIO -> /GPIO01
- J2 pad 4: /GPIO19 -> /GPIO02
- J2 pad 5: /GPIO20 -> /GPIO03
- J2 pad 6: /GPIO21 -> /GPIO04
- J2 pad 7: /GPIO22 -> /GPIO05
- J2 pad 8: /GPIO23 -> /GPIO06
- J2 pad 9: /GPIO24 -> /GPIO07
- J3 pad 1: +3V3 -> /RST
- J3 pad 10: /GPIO10 -> /GPIO25
- J3 pad 11: /GPIO11 -> /GPIO26
- J3 pad 12: /GPIO12 -> /GPIO27
- J3 pad 13: /GPIO13 -> /GPIO28
- J3 pad 14: /GPIO14 -> /GPIO29
- J3 pad 15: /GPIO15 -> GND
- J3 pad 16: GND -> /VSYS
- J3 pad 2: GND -> /SWCLK
- J3 pad 3: /GPIO03 -> /SWDIO
- J3 pad 4: /GPIO04 -> /GPIO19
- J3 pad 5: /GPIO05 -> /GPIO20
- J3 pad 6: /GPIO06 -> /GPIO21
- J3 pad 7: /GPIO07 -> /GPIO22
- J3 pad 8: /GPIO08 -> /GPIO23
- J3 pad 9: /GPIO09 -> /GPIO24
- LED1 pad 1: /GPIO16 -> GND
- LED1 pad 2: Net-(LED1-K) -> /GPIO14
- R7 pad 1: Net-(C10-Pad1) -> Net-(C11-Pad1)
- R8 pad 1: GND -> +3V3
- R8 pad 2: Net-(LED1-K) -> /RST
- U2 pad 1: /D- -> /D+
- U2 pad 2: VBUS -> GND
- U2 pad 3: /D+ -> /D-
- U2 pad 4: /sD+ -> /sD-
- U2 pad 5: GND -> VBUS
- U2 pad 6: /sD- -> /sD+
- U3 pad 1: /VSYS -> GND
- U3 pad 2: GND -> +3V3
- U3 pad 3: +3V3 -> /VSYS
- Y1 pad 3: Net-(C10-Pad1) -> Net-(C11-Pad1)
Routing:
- net +3V3: track 0.00 -> 113.9 mm, vias 0 -> 6
- net GND: track 0.00 -> 95.0 mm, vias 0 -> 30
- net VBUS: track 0.00 -> 28.5 mm, vias 0 -> 4
- net +1V1: track 0.00 -> 26.8 mm, vias 0 -> 2
- net /RST: track 0.00 -> 19.5 mm, vias 0 -> 3
- net /GPIO01: track 0.00 -> 19.2 mm, vias 0 -> 1
- net /GPIO02: track 0.00 -> 18.0 mm, vias 0 -> 1
- net /VSYS: track 0.00 -> 17.8 mm
- net /GPIO03: track 0.00 -> 16.7 mm, vias 0 -> 1
- net /GPIO29: track 0.00 -> 16.7 mm, vias 0 -> 1
- net /GPIO04: track 0.00 -> 16.5 mm, vias 0 -> 1
- net /GPIO05: track 0.00 -> 16.1 mm, vias 0 -> 1
- net /GPIO06: track 0.00 -> 15.7 mm, vias 0 -> 1
- net /Q_SD3: track 0.00 -> 15.6 mm, vias 0 -> 2
- net /GPIO26: track 0.00 -> 15.3 mm, vias 0 -> 1
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- added copper zone on B.Cu, net GND
- added copper zone on F.Cu, net GND
Other:
- board size 23 x 39 mm -> 23 x 35.1 mm
- board text added: "BOOT"
- board text added: "RST"

Commit message: Ready to send off for first fab
Parts:
- J1: footprint Connector_USB:USB_C_Receptacle_HRO_TYPE-C-31-M-12 -> custom:USB_C_Receptacle_HRO_TYPE-C-31-M-12_WITH_3D_MODEL
- R1, R7: footprint Resistor_SMD:R_0402_1005Metric -> Resistor_SMD:R_0805_2012Metric
- moved Y1 1.31 mm to (139.9, 113.5)
- moved C10 1.31 mm to (137.6, 114.7)
- moved C11 1.31 mm to (139.2, 116.3)
- moved R7 0.84 mm to (142.8, 113.7)
- moved R1 0.45 mm to (132.0, 102.0)
- moved C7 0.28 mm to (144.4, 113.0)
- moved C3 0.19 mm to (132.4, 111.0)
- moved D1 0.14 mm to (138.9, 84.0)
Routing:
- net GND: track 95.0 -> 118.3 mm
- net /sD+: track 7.52 -> 6.18 mm
- net /XIN: track 7.01 -> 8.15 mm
- net +3V3: track 113.9 -> 113.0 mm
- net VBUS: track 28.5 -> 27.5 mm
- net /sD-: track 5.98 -> 5.37 mm
- net /RST: track 19.5 -> 19.3 mm, vias 3 -> 2
Other:
- outline, holes or cut-outs redrawn
- board text added: "O"
- board text added: "X"
- board text added: "tctcto v0.1 RevA"
