File: rp2040-board.kicad_sch (KiCad schematic)
At the start: 68 parts, among them CN1 HX JN1.27-2X5 TP H4.9, J1 USB_C_Receptacle_USB2.0_14P, J10 HalfHole, J11 HalfHole, J12 HalfHole, J13 HalfHole, J14 HalfHole, J15 HalfHole, J16 HalfHole, J17 HalfHole, J18 HalfHole, J19 HalfHole, J2 HalfHole, J20 HalfHole, J21 HalfHole, J22 HalfHole, J23 HalfHole, J24 HalfHole, J25 HalfHole, J26 HalfHole, J27 HalfHole, J28 HalfHole, J29 HalfHole, J3 HalfHole, J30 HalfHole, J31 HalfHole, J32 HalfHole, J4 HalfHole, J5 HalfHole, J6 HalfHole, J7 HalfHole, J8 HalfHole, J9 HalfHole, SW1 TS-1088-AR02016, SW2 TS-1088-AR02016, U1 W25Q128JVSIQTR, U2 USBLC6-2SC6, U3 LM3940IMP-3.3/NOPB, U4 RP2040, Y1 ABM8-272-T3_C20625731

Commit message: Working on pcb design
Parts:
- removed D2: LED_Small, symbol Device:LED_Small
- removed J10, J11, J12, J13, J14, J15, J16, J17, J18, J19, J2, J20, J21, J22, J23, J24, J25, J26, J27, J28, J29, J3, J30, J31, J32, J4, J5, J6, J7, J8, J9: HalfHole, symbol Connector:Conn_01x01_Pin
- added J2, J3: (no value), custom:2.0mm_16x1_castellated, symbol custom:2.0mm_16x1_castellated_half_hole
- added LED1: 0603White light_C2290, easyeda2kicad:LED0603-R-RD_WHITE, symbol easyeda2kicad:0603Whitelight_C2290
- C1, C11, C12, C15, C16, C17, C4, C5, C6, C7, C8: footprint (none) -> Capacitor_SMD:C_0402_1005Metric; LCSC Part (none) -> C1525
- C10, C9: footprint (none) -> Capacitor_SMD:C_0402_1005Metric; LCSC Part (none) -> C1548
- C13, C14: footprint (none) -> Capacitor_SMD:C_0402_1005Metric; LCSC Part (none) -> C52923
- C2: footprint (none) -> Capacitor_SMD:C_0402_1005Metric; LCSC Part (none) -> C15525
- C3: footprint (none) -> Capacitor_SMD:C_0603_1608Metric; LCSC Part (none) -> C59461
- J1: footprint (none) -> Connector_USB:USB_C_Receptacle_GCT_USB4105-xx-A_16P_TopMnt_Horizontal; LCSC Part (none) -> C3020560
- R1, R7: footprint (none) -> Resistor_SMD:R_0402_1005Metric; LCSC Part (none) -> C11702
- R2, R9: footprint (none) -> Resistor_SMD:R_0402_1005Metric; LCSC Part (none) -> C60489
- R3, R4: value R_Small -> 5.1Kohm; footprint (none) -> Resistor_SMD:R_0805_2012Metric; LCSC Part (none) -> C27834
- R5, R6: footprint (none) -> Resistor_SMD:R_0603_1608Metric; LCSC Part (none) -> C25190
- R8: value 33Ohm -> 330Ohm; footprint (none) -> Resistor_SMD:R_0603_1608Metric; LCSC Part (none) -> C23138
- U2: LCSC Part (none) -> C7519
- Y1: LCSC Part (none) -> C20625731
Connections:
- net +3V3: now also J3.1
- net GND: now also J2.15, J3.16, J3.2
- net GPIO03: now also J3.3
- net GPIO04: now also J3.4
- net GPIO05: now also J3.5
- net GPIO06: now also J3.6
- net GPIO07: now also J3.7
- net GPIO08: now also J3.8
- net GPIO09: now also J3.9
- net GPIO10: now also J3.10
- net GPIO11: now also J3.11
- net GPIO12: now also J3.12
- net GPIO13: now also J3.13
- net GPIO14: now also J3.14
- net GPIO15: now also J3.15
- net GPIO16: now also LED1.1 (A)
- net GPIO19: now also J2.4
- net GPIO20: now also J2.5
- net GPIO21: now also J2.6
- net GPIO22: now also J2.7
- net GPIO23: now also J2.8
- net GPIO24: now also J2.9
- net GPIO25: now also J2.10
- net GPIO26: now also J2.11
- net GPIO27: now also J2.12
- net GPIO28: now also J2.13
- net GPIO29: now also J2.14
- net RST: now also J2.1
- net SWCLK: now also J2.2
- net SWDIO: now also J2.3
- net VSYS: now also J2.16
- net at R8.2: now also LED1.2 (K)
- no-connect marks 3 -> 6

Commit message: Hopefully finished routing
Parts:
- removed CN1: HX JN1.27-2X5 TP H4.9, easyeda2kicad:IDC-SMD_10P-P1.27-3220-10-0300-00, symbol easyeda2kicad:HXJN1.27-2X5TPH4.9
- removed LED1: 0603White light_C2290, easyeda2kicad:LED0603-R-RD_WHITE, symbol easyeda2kicad:0603Whitelight_C2290
- removed R8: 330Ohm, Resistor_SMD:R_0603_1608Metric, symbol Device:R_Small
- removed U3: LM3940IMP-3.3/NOPB, easyeda2kicad:SOT-223_L6.5-W3.5-P2.30-LS7.0-BR, symbol easyeda2kicad:LM3940IMP-3.3_NOPB
- added C3: 0.1uf, Capacitor_SMD:C_0402_1005Metric, symbol Device:C_Small
- added CN1: SM04B-SRSS-TB, easyeda2kicad:CONN-SMD_4P-P1.00_SM04B-SRSS-TB-LF-SN, symbol easyeda2kicad:SM04B-SRSS-TB
- added LED1: SK6812MINI-E_C5149201, easyeda2kicad:LED-SMD_4P-L3.2-W2.8-LS5.9_SK6812MINI-E, symbol easyeda2kicad:SK6812MINI-E_C5149201
- added U3: AMS1117-3.3, easyeda2kicad:SOT-223-3_L6.5-W3.4-P2.30-LS7.0-BR, symbol easyeda2kicad:AMS1117-3.3
- J1: footprint Connector_USB:USB_C_Receptacle_GCT_USB4105-xx-A_16P_TopMnt_Horizontal -> Connector_USB:USB_C_Receptacle_HRO_TYPE-C-31-M-12; LCSC Part C3020560 -> C165948
- J2: renamed from J3; Exclude from BOM (none) -> 1
- J3: renamed from J2; Exclude from BOM (none) -> 1
- renumbered C9 to C10, C10 to C11, C11 to C12, C12 to C13, C13 to C14, C14 to C15, C15 to C16, C16 to C17, C17 to C18, C3 to C4, C4 to C5, C5 to C6, C6 to C7, C7 to C8, C8 to C9, R9 to R8
Connections:
- net +3V3: now also C3.2, CN1.2, LED1.3 (VDD), U3.2 (VOUT), U3.4 (VOUT)
- net D+: now also U2.1 (I/O1); no longer U2.3 (I/O2)
- net D-: now also U2.3 (I/O2); no longer U2.1 (I/O1)
- net GND: now also U2.2 (GND), C3.1, CN1.1, CN1.5, CN1.6, LED1.1 (GND), U3.1 (GND); no longer U2.5 (VBUS)
- net GPIO01: now also J2.3
- net GPIO02: now also J2.4
- net GPIO03: now also J2.5; no longer J2.3
- net GPIO04: now also J2.6; no longer J2.4
- net GPIO05: now also J2.7; no longer J2.5
- net GPIO06: now also J2.8; no longer J2.6
- net GPIO07: now also J2.9; no longer J2.7
- net GPIO08: now also J2.10; no longer J2.8
- net GPIO09: now also J2.11; no longer J2.9
- net GPIO10: now also J2.12; no longer J2.10
- net GPIO11: now also J2.13; no longer J2.11
- net GPIO12: now also J2.14; no longer J2.12
- net GPIO13: now also J2.15; no longer J2.13
- net GPIO14: now also LED1.2 (DIN); no longer J2.14
- net GPIO15: no longer J2.15
- net GPIO16: now also CN1.3
- net GPIO17: now also CN1.4
- net VBUS: now also U2.5 (VBUS); no longer U2.2 (GND)
- net VSYS: now also U3.3 (VIN)
- net sD+: now also U2.6 (I/O1); no longer U2.4 (I/O2)
- net sD-: now also U2.4 (I/O2); no longer U2.6 (I/O1)
- no-connect marks 6 -> 4
Other:
- note added: "ADC_AVDD/USB_VDD"
- note removed: "ADC_AVDD/USB_AVDD"
- moved on the sheet: C17, C18

Commit message: Ready to send off for first fab
Parts:
- J1: footprint Connector_USB:USB_C_Receptacle_HRO_TYPE-C-31-M-12 -> custom:USB_C_Receptacle_HRO_TYPE-C-31-M-12_WITH_3D_MODEL
Changed lines of the file:
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@@
 			)
 		)
-		(property "Footprint" "Connector_USB:USB_C_Receptacle_HRO_TYPE-C-31-M-12"
+		(property "Footprint" "custom:USB_C_Receptacle_HRO_TYPE-C-31-M-12_WITH_3D_MODEL"
 			(at 203.2 43.18 0)
 			(hide yes)
